File: pcb/cwl/cwl.kicad_sch (KiCad schematic)
At the start: 0 parts

Commit message: new pcb
Parts:
- added D1, D2, D3, D4: 1N4148WS, Diode_SMD:D_SOD-323, symbol Device:D
- added D5: BZT52C4V7, Diode_SMD:D_SOD-123, symbol Device:D_Zener
- added D6: BZT52C15, Diode_SMD:D_SOD-123, symbol Device:D_Zener
- added D7: BZT52C4V3, Diode_SMD:D_SOD-123, symbol Device:D_Zener
- added J1: UEXT, IDC:IDC-Stecker_2x05_P2.54mm_Vertical, symbol Connector_Generic:Conn_02x05_Odd_Even
- added J2: OpenTherm, TerminalBlock_Phoenix:TerminalBlock_Phoenix_MKDS-1,5-2-5.08_1x02_P5.08mm_Horizontal, symbol Connector:Conn_01x02_Pin
- added J3: OLED, SSD1306:128x64OLED-MountingHoles-Combined, symbol Connector:Conn_01x04_Pin
- added LED1: Green, LED_SMD:LED_0805_2012Metric, symbol Device:LED
- added MH1, MH2, MH3, MH4: M3, MountingHole:MountingHole_3.2mm_M3_Pad_Via, symbol Mechanical:MountingHole_Pad
- added Q1: BC858A, Package_TO_SOT_SMD:SOT-23, symbol Transistor_BJT:BC858
- added R1, R4: 330, Resistor_SMD:R_0603_1608Metric, symbol Device:R
- added R2: 220, Resistor_SMD:R_0603_1608Metric, symbol Device:R
- added R3: 100, Resistor_SMD:R_0603_1608Metric, symbol Device:R
- added R5: 1.5k, Resistor_SMD:R_0603_1608Metric, symbol Device:R
- added R6, R7: 10k, Resistor_SMD:R_0603_1608Metric, symbol Device:R
- added R8: 1k, Resistor_SMD:R_0603_1608Metric, symbol Device:R
- added SB3: TXD→OT_TX, Jumper:SolderJumper-2_P1.3mm_Bridged_RoundedPad1.0x1.5mm, symbol Jumper:SolderJumper_2_Bridged
- added SB4: RXD→OT_RX, Jumper:SolderJumper-2_P1.3mm_Bridged_RoundedPad1.0x1.5mm, symbol Jumper:SolderJumper_2_Bridged
- added SW1: EC12E24204A9, Rotary_Encoder:RotaryEncoder_Alps_EC12E-Switch_Vertical_H20mm, symbol Device:RotaryEncoder_Switch
- added U1, U2: PC817, Package_SO:SOP-4_7.5x4.1mm_P2.54mm, symbol Isolator:PC817
Connections:
- new net: D1.1 (K), D2.1 (K), Q1.2 (E), R1.1
- new net: LED1.2 (A), R8.2
- new net: D6.1 (K), Q1.1 (B), R1.2, U1.4
- new net: D3.2 (A), D4.2 (A), D5.2 (A), D6.2 (A), D7.2 (A), R3.2, U2.2
- new net: R4.1, U1.1
- new net: D7.1 (K), U1.3
- new net: R2.1, R3.1, U2.1
- new net: D5.1 (K), Q1.3 (C), R2.2
- new net +3V3: J1.1 (Pin_1), J3.1 (Pin_1), R6.1, R7.2, U2.4
- new net ENC_CLK: J1.7 (Pin_7), R6.2, SW1.A
- new net ENC_DT: J1.9 (Pin_9), R7.1, SW1.B
- new net ENC_SW: J1.10 (Pin_10), SW1.S1
- new net GND: J1.2 (Pin_2), J3.2 (Pin_2), LED1.1 (K), MH1.1, MH2.1, MH3.1, MH4.1, R5.2, SW1.C, SW1.S2, U1.2
- new net LED_GPIO: J1.8 (Pin_8), R8.1
- new net OT+: D1.2 (A), D3.1 (K), J2.2 (Pin_2)
- new net OT-: D2.2 (A), D4.1 (K), J2.1 (Pin_1)
- new net OT_RX_SIG: R5.1, SB4.2 (B), U2.3
- new net OT_TX_SIG: R4.2, SB3.2 (B)
- new net SCL: J1.5 (Pin_5), J3.3 (Pin_3)
- new net SDA: J1.6 (Pin_6), J3.4 (Pin_4)
- new net UEXT_RXD: J1.4 (Pin_4), SB4.1 (A)
- new net UEXT_TXD: J1.3 (Pin_3), SB3.1 (A)
Other:
- note added: "Display / LED"
- note added: "Encoder"
- note added: "OpenTherm"
- note added: "UEXT"
- title: (none) -> SKiDL-Generated Schematic

Commit message: new pcb
Parts:
- renumbered SB3 to SB1, SB4 to SB2
Other:
- moved on the sheet: SB1, SB2
Changed lines of the file:
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@@
 	(global_label "UEXT_RXD"
 		(shape bidirectional)
-		(at 326.39 97.79 180)
+		(at 326.39 96.52 180)
 		(effects
 			(font
@@
 		)
 		(property "Intersheetrefs" "${INTERSHEET_REFS}"
-			(at 326.39 97.79 0)
+			(at 326.39 96.52 0)
 			(hide yes)
 			(show_name no)
@@
 	(global_label "OT_TX_SIG"
 		(shape bidirectional)
-		(at 336.55 105.41 0)
+		(at 336.55 107.95 0)
 		(effects
 			(font
@@
 		)
 		(property "Intersheetrefs" "${INTERSHEET_REFS}"
-			(at 336.55 105.41 0)
+			(at 336.55 107.95 0)
 			(hide yes)
 			(show_name no)
@@
 	(global_label "UEXT_TXD"
 		(shape bidirectional)
-		(at 326.39 105.41 180)
+		(at 326.39 107.95 180)
 		(effects
 			(font
@@
 		)
 		(property "Intersheetrefs" "${INTERSHEET_REFS}"
-			(at 326.39 105.41 0)
+			(at 326.39 107.95 0)
 			(hide yes)
 			(show_name no)
@@
 	(global_label "OT_RX_SIG"
 		(shape bidirectional)
-		(at 336.55 97.79 0)
+		(at 336.55 96.52 0)
 		(effects
 			(font
@@
 		)
 		(property "Intersheetrefs" "${INTERSHEET_REFS}"
-			(at 336.55 97.79 0)
+			(at 336.55 96.52 0)
 			(hide yes)
 			(show_name no)
@@
 	(symbol
 		(lib_id "Jumper:SolderJumper_2_Bridged")
-		(at 331.47 97.79 0)
+		(at 331.47 96.52 0)
 		(unit 1)
 		(body_style 1)
@@
 		(dnp no)
 		(fields_autoplaced yes)
-		(property "Reference" "SB4"
-			(at 331.47 95.25 0)
-			(show_name no)
-			(do_not_autoplace no)
-			(effects
-				(font
-					(size 1.27 1.27)
-				)
-				(justify left)
+		(property "Reference" "SB2"
+			(at 331.47 90.17 0)
+			(show_name no)
+			(do_not_autoplace no)
+			(effects
+				(font
+					(size 1.27 1.27)
+				)
 			)
 		)
 		(property "Value" "RXD→OT_RX"
-			(at 331.47 100.33 0)
-			(show_name no)
-			(do_not_autoplace no)
-			(effects
-				(font
-					(size 1.27 1.27)
-				)
-				(justify left)
+			(at 331.47 92.71 0)
+			(show_name no)
+			(do_not_autoplace no)
+			(effects
+				(font
+					(size 1.27 1.27)
+				)
 			)
 		)
 		(property "Footprint" "Jumper:SolderJumper-2_P1.3mm_Bridged_RoundedPad1.0x1.5mm"
-			(at 331.47 97.79 0)
+			(at 331.47 96.52 0)
 			(hide yes)
 			(show_name no)
@@
 		)
 		(property "Datasheet" ""
-			(at 331.47 97.79 0)
+			(at 331.47 96.52 0)
 			(hide yes)
 			(show_name no)
@@
 		)
 		(property "Description" "Solder Jumper, 2-pole, closed/bridged"
-			(at 331.47 97.79 0)
+			(at 331.47 96.52 0)
 			(hide yes)
 			(show_name no)
@@
 			(project "cwl"
 				(path "/218b5f90-a139-55d3-a988-331ecbe7ee0c"
-					(reference "SB4")
+					(reference "SB2")
 					(unit 1)
 				)
@@
 	(symbol
 		(lib_id "Jumper:SolderJumper_2_Bridged")
-		(at 331.47 105.41 0)
+		(at 331.47 107.95 0)
 		(unit 1)
 		(body_style 1)
@@
 		(dnp no)
 		(fields_autoplaced yes)
-		(property "Reference" "SB3"
-			(at 331.47 102.87 0)
-			(show_name no)
-			(do_not_autoplace no)
-			(effects
-				(font
-					(size 1.27 1.27)
-				)
-				(justify left)
+		(property "Reference" "SB1"
+			(at 331.47 101.6 0)
+			(show_name no)
+			(do_not_autoplace no)
+			(effects
+				(font
+					(size 1.27 1.27)
+				)
 			)
 		)
 		(property "Value" "TXD→OT_TX"
+			(at 331.47 104.14 0)
+			(show_name no)
+			(do_not_autoplace no)
+			(effects
+				(font
+					(size 1.27 1.27)
+				)
+			)
+		)
+		(property "Footprint" "Jumper:SolderJumper-2_P1.3mm_Bridged_RoundedPad1.0x1.5mm"
 			(at 331.47 107.95 0)
-			(show_name no)
-			(do_not_autoplace no)
-			(effects
-				(font
-					(size 1.27 1.27)
-				)
-				(justify left)
-			)
-		)
-		(property "Footprint" "Jumper:SolderJumper-2_P1.3mm_Bridged_RoundedPad1.0x1.5mm"
-			(at 331.47 105.41 0)
 			(hide yes)
 			(show_name no)
@@
 		)
 		(property "Datasheet" ""
-			(at 331.47 105.41 0)
+			(at 331.47 107.95 0)
 			(hide yes)
 			(show_name no)
@@
 		)
 		(property "Description" "Solder Jumper, 2-pole, closed/bridged"
-			(at 331.47 105.41 0)
+			(at 331.47 107.95 0)
 			(hide yes)
 			(show_name no)
@@
 			(project "cwl"
 				(path "/218b5f90-a139-55d3-a988-331ecbe7ee0c"
-					(reference "SB3")
+					(reference "SB1")
 					(unit 1)
 				)
