File: pcb/cwl-diyless/cwl.kicad_pcb (KiCad board)
At the start: 2 copper layers, 107.7 x 56.9 mm, 14 parts, among them J1 UEXT, J3 OLED_0.96, J3B OLED_1.3, J6 D1mini, J8 UEXT_DBG, SW1 EC12E24204A9

Commit message: new pcb
Other:
- board text added: "philipparndt/opentherm-wolf-cwl DIYless 2026-05-17 v0.2.0"
- board text removed: "philipparndt/opentherm-wolf-cwl 2026-05-16 v0.2.0"
Changed lines of the file:
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@@
 		(layer "Edge.Cuts")
 	)
-	(gr_text "philipparndt/opentherm-wolf-cwl\n2026-05-16 v0.2.0"
-		(at 83.05 83.76 0)
+	(gr_text "philipparndt/opentherm-wolf-cwl DIYless\n2026-05-17 v0.2.0"
+		(at 82.6 80.28 0)
 		(layer "F.SilkS")
 		(effects

Commit message: new pcb
Parts:
- removed the J3 at (140.1, 72.2)
- J3B: footprint SSD1306:128x64OLED-MountingHoles-Large -> SSD1306:128x64OLED-MountingHoles-Combined
- moved J3B 1.55 mm to (108.6, 41.0)
- renumbered J6 to J2, J8 to J3
Routing:
- net GND: track 322.7 -> 336.0 mm, vias 4 -> 6
- net +3V3: track 119.1 -> 113.3 mm, vias 2 -> 1
- net OT_RX_SIG: track 114.1 -> 115.1 mm
- net SCL: track 50.5 -> 51.4 mm
Other:
- board text added: "RoHS Compliant"
