File: pcb/cwl-compact/cwl.kicad_pcb (KiCad board)
At the start: 2 copper layers, 100 x 70 mm, 29 parts, among them J1 UEXT, J2 OpenTherm, J3 OLED, Q1 BC858A, SW1 EC12E24204A9, U1 PC817, U2 PC817

Commit message: history page + tz
Parts:
- moved J1 6.15 mm to (85.2, 111.9)
- moved D1 5.00 mm to (52.9, 101.1)
- moved D2 5.00 mm to (52.9, 106.7)
- moved D3 5.00 mm to (52.9, 103.9)
- moved D4 5.00 mm to (52.9, 109.5)
- moved D5 5.00 mm to (64.7, 108.3)
- moved D6 5.00 mm to (64.7, 105.1)
- moved D7 5.00 mm to (64.7, 101.9)
- moved J2 5.00 mm to (38.9, 102.6)
- moved MH2 5.00 mm to (36.4, 117.0)
- moved Q1 5.00 mm to (58.1, 105.1)
- moved R1 5.00 mm to (58.1, 101.2)
- moved R2 5.00 mm to (58.1, 108.8)
- moved R3 5.00 mm to (58.1, 110.8)
- moved R4 5.00 mm to (62.4, 94.4)
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Routing:
- net GND: track 306.0 -> 406.8 mm, vias 2 -> 5
- net +3V3: track 200.0 -> 179.3 mm
- net ENC_CLK: track 65.5 -> 59.7 mm
- net LED_GPIO: track 69.5 -> 74.9 mm
- net UEXT_TXD: track 27.0 -> 22.5 mm
- net SCL: track 65.3 -> 60.9 mm
- net UEXT_RXD: track 22.7 -> 18.9 mm
- net SDA: track 60.4 -> 57.8 mm
- net ENC_SW: track 44.7 -> 42.9 mm
- net ENC_DT: track 58.4 -> 57.6 mm
Other:
- board size 100 x 70 mm -> 100 x 65 mm
- board text added: "philipparndt/opentherm-wolf-cwl 2026-05-25 v0.3.0"
- board text removed: "philipparndt/opentherm-wolf-cwl 2026-05-17 v0.3.0"
